File: DAC-ADC SPI module/DAC-ADC SPI module.sch (KiCad schematic (older format))
At the start: 14 parts

Commit message: Schematic capture completed
Parts:
- C1, C2: renamed from C?; value 2.2uF -> 2.2u
- C3, C5: renamed from C?; value 0.1uF -> 0.1u
- C4, C6: renamed from C?; value 10uF -> 10u
- gave numbers to parts that had none: 8
Connections:
- wire segments 87 -> 90
Other:
- moved on the sheet: C3, C4, J2

Commit message: PCB layout complete
Parts:
- removed J2: Conn_01x02_Male, symbol Connector:Conn_01x02_Male
- removed J3: Conn_01x06_Male, symbol Connector:Conn_01x06_Male
- added J2: Conn_01x08_Male, Pin_Headers:Pin_Header_Straight_1x08_Pitch2.54mm, symbol Connector:Conn_01x08_Male
- C1, C2, C3, C4, C5, C6: footprint (none) -> Capacitors_SMD:C_0805_HandSoldering
- J1: footprint (none) -> Pin_Headers:Pin_Header_Straight_1x04_Pitch2.54mm
- J4: footprint (none) -> Pin_Headers:Pin_Header_Straight_1x02_Pitch2.54mm
- R1: footprint (none) -> Resistors_SMD:R_0805_HandSoldering
- U1, U3: footprint (none) -> SMD_Packages:SOIC-8-N
- U2: footprint (none) -> SMD_Packages:SOIC-14_N
Connections:
- wire segments 90 -> 88
Changed lines of the file:
@@
 F 0 "U2" H 5185 4050 50  0000 C CNN
 F 1 "MCP3204" H 5310 3975 50  0000 C CNN
-F 2 "" H 6000 3300 50  0001 C CNN
+F 2 "SMD_Packages:SOIC-14_N" H 6000 3300 50  0001 C CNN
 F 3 "http://ww1.microchip.com/downloads/en/DeviceDoc/21298c.pdf" H 6000 3300 50  0001 C CNN
 	1    5100 3600
@@
 F 0 "U1" H 3480 2895 50  0000 C CNN
 F 1 "MCP1501" H 3610 2825 50  0000 C CNN
-F 2 "" H 4600 2100 50  0001 C CIN
+F 2 "SMD_Packages:SOIC-8-N" H 4600 2100 50  0001 C CIN
 F 3 "https://ww1.microchip.com/downloads/en/DeviceDoc/20005474E.pdf" H 3500 2150 50  0001 C CIN
 	1    3400 2550
@@
 F 0 "U3" H 6985 4045 50  0000 C CNN
 F 1 "MCP4822" H 7110 3975 50  0000 C CNN
-F 2 "" H 7700 3300 50  0001 C CNN
+F 2 "SMD_Packages:SOIC-8-N" H 7700 3300 50  0001 C CNN
 F 3 "http://ww1.microchip.com/downloads/en/DeviceDoc/20002249B.pdf" H 7700 3300 50  0001 C CNN
 	1    6900 3600
@@
 F 0 "J1" H 1903 3789 50  0000 C CNN
 F 1 "Conn_01x04_Male" H 1903 3790 50  0001 C CNN
-F 2 "" H 1795 3600 50  0001 C CNN
+F 2 "Pin_Headers:Pin_Header_Straight_1x04_Pitch2.54mm" H 1795 3600 50  0001 C CNN
 F 3 "~" H 1795 3600 50  0001 C CNN
 	1    1795 3600
@@
 Wire Wire Line
 	4500 3800 1995 3800
-$Comp
-L Connector:Conn_01x06_Male J3
-U 1 1 606B10DA
-P 1800 4900
-F 0 "J3" H 1908 5189 50  0000 C CNN
-F 1 "Conn_01x06_Male" H 1908 5190 50  0001 C CNN
-F 2 "" H 1800 4900 50  0001 C CNN
-F 3 "~" H 1800 4900 50  0001 C CNN
-	1    1800 4900
-	1    0    0    -1
-$EndComp
 Entry Wire Line
 	2400 4700 2500 4600
@@
 F 0 "J4" H 8172 3528 50  0000 R CNN
 F 1 "Conn_01x02_Male" H 8172 3573 50  0001 R CNN
-F 2 "" H 8200 3600 50  0001 C CNN
+F 2 "Pin_Headers:Pin_Header_Straight_1x02_Pitch2.54mm" H 8200 3600 50  0001 C CNN
 F 3 "~" H 8200 3600 50  0001 C CNN
 	1    8200 3600
@@
 L power:+5V #PWR04
 U 1 1 606CAD81
-P 4000 1850
-F 0 "#PWR04" H 4000 1700 50  0001 C CNN
-F 1 "+5V" H 4015 2023 50  0000 C CNN
-F 2 "" H 4000 1850 50  0001 C CNN
-F 3 "" H 4000 1850 50  0001 C CNN
-	1    4000 1850
-	1    0    0    -1
-$EndComp
-Wire Wire Line
-	4000 1850 4000 1950
+P 4000 1800
+F 0 "#PWR04" H 4000 1650 50  0001 C CNN
+F 1 "+5V" H 4015 1973 50  0000 C CNN
+F 2 "" H 4000 1800 50  0001 C CNN
+F 3 "" H 4000 1800 50  0001 C CNN
+	1    4000 1800
+	1    0    0    -1
+$EndComp
+Wire Wire Line
+	4000 1800 4000 1850
 Connection ~ 4000 1950
 Wire Wire Line
@@
 Wire Wire Line
 	6900 4200 6900 4100
-$Comp
-L Connector:Conn_01x02_Male J2
-U 1 1 606CF058
-P 1800 1950
-F 0 "J2" H 1908 2039 50  0000 C CNN
-F 1 "Conn_01x02_Male" H 1908 2040 50  0001 C CNN
-F 2 "" H 1800 1950 50  0001 C CNN
-F 3 "~" H 1800 1950 50  0001 C CNN
-	1    1800 1950
-	1    0    0    -1
-$EndComp
-Connection ~ 2950 1950
-$Comp
-L power:GND #PWR01
-U 1 1 606D4166
-P 2050 2100
-F 0 "#PWR01" H 2050 1850 50  0001 C CNN
-F 1 "GND" H 2055 1927 50  0000 C CNN
-F 2 "" H 2050 2100 50  0001 C CNN
-F 3 "" H 2050 2100 50  0001 C CNN
-	1    2050 2100
-	1    0    0    -1
-$EndComp
-Wire Wire Line
-	2000 2050 2050 2050
-Wire Wire Line
-	2050 2050 2050 2100
-Text Label 2050 1950 0    50   ~ 0
+Text Label 4050 1950 0    50   ~ 0
 VDD
 Wire Wire Line
@@
 F 0 "C2" H 4342 3046 50  0000 L CNN
 F 1 "2.2u" H 4342 2955 50  0000 L CNN
-F 2 "" H 4250 3000 50  0001 C CNN
+F 2 "Capacitors_SMD:C_0805_HandSoldering" H 4250 3000 50  0001 C CNN
 F 3 "~" H 4250 3000 50  0001 C CNN
 	1    4250 3000
@@
 F 0 "C1" V 3740 2195 50  0000 C CNN
 F 1 "2.2u" V 3745 1970 50  0000 C CNN
-F 2 "" H 3700 2100 50  0001 C CNN
+F 2 "Capacitors_SMD:C_0805_HandSoldering" H 3700 2100 50  0001 C CNN
 F 3 "~" H 3700 2100 50  0001 C CNN
 	1    3700 2100
@@
 F 0 "R1" H 4318 2746 50  0000 L CNN
 F 1 "50R" H 4318 2655 50  0000 L CNN
-F 2 "" H 4250 2700 50  0001 C CNN
+F 2 "Resistors_SMD:R_0805_HandSoldering" H 4250 2700 50  0001 C CNN
 F 3 "~" H 4250 2700 50  0001 C CNN
 	1    4250 2700
@@
 F 0 "C5" H 7192 2696 50  0000 L CNN
 F 1 "0.1u" H 7192 2605 50  0000 L CNN
-F 2 "" H 7100 2650 50  0001 C CNN
+F 2 "Capacitors_SMD:C_0805_HandSoldering" H 7100 2650 50  0001 C CNN
 F 3 "~" H 7100 2650 50  0001 C CNN
 	1    7100 2650
@@
 F 0 "C6" H 7592 2696 50  0000 L CNN
 F 1 "10u" H 7592 2605 50  0000 L CNN
-F 2 "" H 7500 2650 50  0001 C CNN
+F 2 "Capacitors_SMD:C_0805_HandSoldering" H 7500 2650 50  0001 C CNN
 F 3 "~" H 7500 2650 50  0001 C CNN
 	1    7500 2650
@@
 F 0 "C3" H 5392 2696 50  0000 L CNN
 F 1 "0.1u" H 5392 2605 50  0000 L CNN
-F 2 "" H 5300 2650 50  0001 C CNN
+F 2 "Capacitors_SMD:C_0805_HandSoldering" H 5300 2650 50  0001 C CNN
 F 3 "~" H 5300 2650 50  0001 C CNN
 	1    5300 2650
@@
 Wire Wire Line
 	6900 2350 6900 3200
-Wire Wire Line
-	2000 1950 2300 1950
 $Comp
 L Device:C_Small C4
@@
 F 0 "C4" H 5792 2696 50  0000 L CNN
 F 1 "10u" H 5792 2605 50  0000 L CNN
-F 2 "" H 5700 2650 50  0001 C CNN
+F 2 "Capacitors_SMD:C_0805_HandSoldering" H 5700 2650 50  0001 C CNN
 F 3 "~" H 5700 2650 50  0001 C CNN
 	1    5700 2650
@@
 L power:PWR_FLAG #FLG0101
 U 1 1 6076D766
-P 2300 1900
-F 0 "#FLG0101" H 2300 1975 50  0001 C CNN
-F 1 "PWR_FLAG" H 2300 2073 50  0000 C CNN
-F 2 "" H 2300 1900 50  0001 C CNN
-F 3 "~" H 2300 1900 50  0001 C CNN
-	1    2300 1900
-	1    0    0    -1
+P 4000 1850
+F 0 "#FLG0101" H 4000 1925 50  0001 C CNN
+F 1 "PWR_FLAG" V 4000 1977 50  0000 L CNN
+F 2 "" H 4000 1850 50  0001 C CNN
+F 3 "~" H 4000 1850 50  0001 C CNN
+	1    4000 1850
+	0    -1   -1   0
 $EndComp
 $Comp
 L power:PWR_FLAG #FLG0102
 U 1 1 6076E3A2
-P 2100 2050
-F 0 "#FLG0102" H 2100 2125 50  0001 C CNN
-F 1 "PWR_FLAG" V 2100 2178 50  0000 L CNN
-F 2 "" H 2100 2050 50  0001 C CNN
-F 3 "~" H 2100 2050 50  0001 C CNN
-	1    2100 2050
+P 2100 5450
+F 0 "#FLG0102" H 2100 5525 50  0001 C CNN
+F 1 "PWR_FLAG" H 2100 5623 50  0000 C CNN
+F 2 "" H 2100 5450 50  0001 C CNN
+F 3 "~" H 2100 5450 50  0001 C CNN
+	1    2100 5450
+	-1   0    0    1
+$EndComp
+$Comp
+L Connector:Conn_01x08_Male J2
+U 1 1 60779499
+P 1800 5000
+F 0 "J2" H 1908 5389 50  0000 C CNN
+F 1 "Conn_01x08_Male" H 1908 5390 50  0001 C CNN
+F 2 "Pin_Headers:Pin_Header_Straight_1x08_Pitch2.54mm" H 1800 5000 50  0001 C CNN
+F 3 "~" H 1800 5000 50  0001 C CNN
+	1    1800 5000
+	1    0    0    -1
+$EndComp
+$Comp
+L power:+5V #PWR0101
+U 1 1 6077F2EE
+P 2250 5300
+F 0 "#PWR0101" H 2250 5150 50  0001 C CNN
+F 1 "+5V" H 2265 5473 50  0000 C CNN
+F 2 "" H 2250 5300 50  0001 C CNN
+F 3 "" H 2250 5300 50  0001 C CNN
+	1    2250 5300
 	0    1    1    0
 $EndComp
-Wire Wire Line
-	2100 2050 2050 2050
-Connection ~ 2050 2050
-Wire Wire Line
-	2300 1900 2300 1950
+$Comp
+L power:GND #PWR0102
+U 1 1 607812A4
+P 2100 5400
+F 0 "#PWR0102" H 2100 5150 50  0001 C CNN
+F 1 "GND" H 2105 5227 50  0000 C CNN
+F 2 "" H 2100 5400 50  0001 C CNN
+F 3 "" H 2100 5400 50  0001 C CNN
+	1    2100 5400
+	0    -1   -1   0
+$EndComp
+Wire Wire Line
+	2000 5400 2100 5400
+Wire Wire Line
+	2100 5400 2100 5450
+Wire Wire Line
+	2000 5300 2250 5300
+Connection ~ 4000 1850
+Wire Wire Line
+	4000 1850 4000 1950
 Wire Bus Line
 	6050 3600 6050 4500
 Wire Bus Line
 	2500 4500 2500 5100
-Connection ~ 2300 1950
-Wire Wire Line
-	2300 1950 2950 1950
+Connection ~ 2100 5400
 $EndSCHEMATC
